File: Eagle/Embedded/NodeBoard/NodeBoard.brd (EAGLE design)
At the start: 121 x 96 mm, 68 parts, among them IC1 7812TV, IC2 5v, IC3 3v3, IC4 REG1117, IC5 REG1117, J1 DCJ0202, Q2 IRF740, T1 BC547

Commit message: Report, and eagle changes
Parts:
- removed C4: 0u33, resistor:E2,5-6E
- removed IC2: 5v, v-reg:317TS
- removed IC3: 3v3, v-reg:317TS
- removed JMP4: 0R-JUMPA, jump-0r-smd:A0R-JMP
- removed JP1: (no value), jumper:JP1
- removed LED3: (no value), adafruit:CHIPLED_1206
- removed LED5: RED, led:LED5MM
- removed MODE_SEL: (no value), special:EDG-04
- removed PLD: VT23N2, photo-elements:TO46-VT200
- removed R11: 160, resistor:R0603
- removed R13: 160, rcl:0204/7
- removed R3, R4, R5: 10k, rcl:0204/7
- added D5, D6: 1N4004, adafruit:DO41-10
- added JP10, JP8, JP9: (no value), jumper:JP4
- added LM317: 3v3, v-reg:317TS
- added LM317T: 5v, v-reg:317TS
- added Q1, Q3: IRF740, transistor-power:TO220BV
- added R21: 1k, rcl:0204/7
- added SD_CARD: (no value), con-lstb:MA06-1
- added T2: BC547, transistor:TO92
- added U$4: RELAY, relay:RELAY
- added X3, X5, X6: (no value), con-wago-500:W237-103
- added X4: (no value), con-wago-500:W237-102
- JP2: device jumper:JP2 -> jumper:JP4
- JP5: device jumper:JP2 -> jumper:JP1
- R1: device rcl:0204/7 -> resistor:R0603
- R2: value (none) -> 10k; device rcl:0204/7 -> resistor:R0603
- U$1: device RELAY:RELAY -> relay:RELAY
- X1: device con-wago-500:W237-6 -> con-wago-500:W237-102
- moved X1 244.3 mm to (122.8, 94.5), flipped to the top, turned to 0 degrees
- moved C7 211.5 mm to (89.6, 16.9), turned to 0 degrees
- moved C8 210.0 mm to (98.0, 11.7)
- moved R17 209.8 mm to (111.8, 16.0), turned to 270 degrees
- moved IC5 209.1 mm to (87.3, 24.3)
- moved C6 208.2 mm to (92.7, 21.9)
- moved JMP8 207.6 mm to (96.3, 20.6)
- moved R15 206.2 mm to (109.5, 15.9), turned to 90 degrees
- moved D2 204.0 mm to (128.2, 31.3), turned to 0 degrees
- moved JP5 200.3 mm to (129.4, 69.6), turned to 0 degrees
- moved C9 200.3 mm to (88.2, 11.8)
- moved R6 199.6 mm to (131.2, 56.8)
- moved R19 199.3 mm to (132.3, 69.6)
- moved DHT 196.6 mm to (135.1, 56.8), turned to 90 degrees
- moved JP3 195.6 mm to (112.2, 25.4), turned to 0 degrees
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Connections:
- net N$12 renamed TX
- net N$13 renamed RX
- net N$15 renamed GPIO12
- removed net N$14: MODE_SEL.6, R5.2, U1.GPIO4
- removed net N$16: MODE_SEL.8, R4.2, U1.GPIO15
- removed net N$21: JP1.1, U1.GPIO16
- removed net N$25: JP5.3, PLD.1, R2.2
- removed net N$26: U$1.COM, X1.1
- removed net N$27: JP2.2, U1.GPIO14
- removed net N$29: JP1.2, R8.1, U$5.2, U1.RESET
- removed net N$3: JP5.2, U1.ADC
- removed net N$32: LED3.A, R11.2
- removed net N$34: LED5.A, R13.1
- removed net N$35: JMP3.2, U1.GPIO10
- removed net N$38: JMP4.2, U1.GPIO13
- removed net N$39: JMP4.3, R11.1
- removed net N$40: JMP4.1, R13.2
- removed net N$59: JP2.1, Q2.G
- removed net N$6: U$1.COM_CPEN, U$2.7, U$3.P$2
- removed net N$7: X1.3, X1.4
- new net 12V_IN: D6.A, J1.1, X1.2, X2.2, X4.2
- new net AC_C: U$2.1, X3.2, X6.1, X6.2
- new net AC_G: X3.1, X5.1, X6.3
- new net AC_P: U$1.COM_CPEN, U$2.7, U$3.P$2, U$4.COM_CPEN
- new net ADC: MQ.4, R19.2, U1.ADC
- new net CS: SD_CARD.5, U1.CS0
- new net GPIO0: Q2.G, R9.1, U$6.1, U1.GPIO0
- new net GPIO10: JP9.4, U1.GPIO10
- new net GPIO13: JP10.4, U1.GPIO13
- new net GPIO14: JP8.4, U1.GPIO14
- new net GPIO15: Q1.G, R1.2, U1.GPIO15
- new net GPIO16: JP2.4, U1.GPIO16
- new net GPIO2: Q3.G, R2.2, U1.GPIO2
- new net GPIO4: R21.2, U1.GPIO4
- new net GPIO5: R14.2, U1.GPIO5
- new net GPIO9: JMP3.2, U1.GPIO9
- new net MISO: SD_CARD.2, U1.MISO
- new net MOSI: SD_CARD.4, U1.MOSI
- new net RST: R8.1, U$5.2, U1.RESET
- new net SCLK: SD_CARD.3, U1.SCLK
- net 12V: now also D6.C; no longer J1.1, X2.2
- net 19V: no longer C4.+
- net 3V3: now also JP10.2, JP2.2, JP8.2, JP9.2, MQ.1, R2.1, SD_CARD.6; no longer MODE_SEL.1, MODE_SEL.2, MODE_SEL.3, MODE_SEL.4
- net GND: now also JP10.3, JP2.3, JP8.3, JP9.3, Q1.S, Q3.S, SD_CARD.1, T2.1; no longer C4.-, LED3.C, LED5.K, R2.1, R3.1, R4.1, R5.1
- net N$18: now also Q1.D, X1.1; no longer MODE_SEL.5, R3.2, U1.GPIO5
- net N$22: now also Q3.D, X4.1; no longer U$6.2, U1.GPIO0
- net N$44: now also R21.1, T2.2; no longer JP2.3, R14.2
- net N$45: now also LM317T.2; no longer IC2.2
- net N$46: now also LM317T.1; no longer IC2.1
- net N$47: now also LM317.2; no longer IC3.2
- net N$48: now also LM317.1; no longer IC3.1
- net N$49: now also LM317T.3; no longer IC2.3
- net N$50: now also LM317.3; no longer IC3.3
- net N$60: now also D5.A, T2.3, U$4.P$2; no longer MODE_SEL.7, R1.2, U1.GPIO2
- net N$62: now also X3.3; no longer X1.6
- net N$63: now also U$4.COM, X5.2; no longer R9.1, U$6.1
- net N$8: now also U$1.COM, X5.3; no longer U$2.1, X1.2, X1.5
- net N$9: now also JP5.2, MQ.3; no longer JP5.1, MQ.4, R19.2
- net VCC: now also D5.C, JP10.1, JP2.1, JP5.1, JP8.1, JP9.1, U$4.P$1; no longer MQ.1, PLD.2
Routing:
- net N$42: track 163.4 -> 42.5 mm, vias 2 -> 0
- net N$26: track 91.8 -> 0.00 mm
- net GPIO9: track 0.00 -> 91.2 mm, vias 0 -> 2
- net AC_G: track 0.00 -> 89.2 mm
- net AC_C: track 0.00 -> 86.5 mm
- net 12V: track 114.2 -> 186.0 mm, vias 1 -> 3
- net 19V: track 106.2 -> 34.7 mm
- net N$38: track 67.4 -> 0.00 mm, vias 2 -> 0
- net AC_P: track 0.00 -> 57.5 mm
- net GPIO2: track 0.00 -> 56.0 mm, vias 0 -> 2
- net N$29: track 56.0 -> 0.00 mm, vias 1 -> 0
- net N$9: track 61.2 -> 5.87 mm
- net 12V_IN: track 0.00 -> 54.8 mm
- net GPIO0: track 0.00 -> 54.0 mm, vias 0 -> 1
- net ADC: track 0.00 -> 52.8 mm, vias 0 -> 1
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Other:
- board size 121 x 96 mm -> 140 x 100 mm
- board text added: "V3.0"
- board text removed: "V2.0"
